File: Servo Driver Board/Servo Driver Board.kicad_sch (KiCad schematic)
At the start: 7 parts, among them J1 Conn_01x05_Pin, J4 Conn_01x04_Pin, U1 ATtiny412-SS, U3 XC6206PxxxMR

Commit message: Exported
Other:
- company: (none) -> Privat
- title: (none) -> Advanced Servo Controller
Changed lines of the file:
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@@
 	(generator_version "9.0")
 	(paper "A4")
+	(title_block
+		(title "Advanced Servo Controller")
+		(rev "1")
+		(company "Privat")
+		(comment 1 "Tristan Wieczorek")
+	)
 	(text "IPROPI μA = Iout(A) * 1500 μA/A\n4A * 1500μA/A = 6000μA\n3,3V / 0,006A = 550R"
 		(exclude_from_sim no)
@@
 		)
 		(property "Footprint" "Resistor_SMD:R_0603_1608Metric"
-			(at 152.4 114.554 90)
-			(effects
-				(font
+			(at 152.4 116.078 90)
+			(effects
+				(font
